Commit message: slam files

File: description/robot.urdf.xacro (robot description, xacro)
@@ -2,3 +2,7 @@
 <robot xmlns:xacro="http://www.ros.org/wiki/xacro"  name="robot">
     <xacro:include filename = "robot_core.xacro"/>
+    <xacro:include filename = "gazebo_control.xacro"/>
+    <xacro:include filename = "lidar.xacro"/>
+    <!-- <xacro:include filename = "camera.xacro"/> -->
+    <xacro:include filename = "depth_camera.xacro"/>
 </robot>

File: description/robot_core.xacro (robot description, xacro)
@@ -2,49 +2,60 @@
 <robot xmlns:xacro="http://www.ros.org/wiki/xacro" >
     <xacro:include filename="inertial_macros.xacro"/>
-    <material name ="white">
-        <color rgba="1.0 1.0 1.0 1.0"/>
+    <material name="white">
+        <color rgba="1 1 1 1" />
     </material>
-    <material name = "orange">
-        <color rgba="1.0 0.3 0.1 1.0"/>
+    <material name="orange">
+        <color rgba="1 0.3 0.1 1"/>
     </material>
-    <material name = "blue">
-        <color rgba="0.2 0.2 1.0 1.0"/>
+    <material name="blue">
+        <color rgba="0.2 0.2 1 1"/>
     </material>
-    <material name = "black">
-        <color rgba="0.0 0.0 0.0 1.0"/>
+    <material name="black">
+        <color rgba="0 0 0 1"/>
     </material>
-    <!-- Base libk-->
+    <!-- BASE LINK -->
     <link name="base_link">
     </link>
-    <!-- Chassis link-->
+    <!--BASE_Footprint_Link-->
+    <joint name="base_footprint_jont" type="fixed">
+        <parent link="base_link"/>
+        <child link="base_footprint"/>
+        <origin xyz="0 0 0" rpy="0 0 0"/>
+    </joint>
+    <link name="base_footprint">
+    </link>
+    <!-- CHASSIS LINK -->
     <joint name="chassis_joint" type="fixed">
         <parent link="base_link"/>
         <child link="chassis"/>
-        <origin xyz="-0.1 0.0 0.0" />
+        <origin xyz="-0.1 0 0"/>
     </joint>
-    <link name= "chassis">
+    <link name="chassis">
         <visual>
-            <origin xyz="0.15 0.0 0.075"/>
+            <origin xyz="0.15 0 0.075"/>
             <geometry>
                 <box size="0.3 0.3 0.15"/>
             </geometry>
-            <material name ="white"/>
+            <material name="white"/>
         </visual>
         <collision>
-            <origin xyz="0.15 0.0 0.075"/>
+            <origin xyz="0.15 0 0.075"/>
             <geometry>
                 <box size="0.3 0.3 0.15"/>
             </geometry>
         </collision>
-        <xacro:inertial_box mass = "0.5" x="0.3" y="0.3" z="0.15">
-            <origin xyz="0.15 0.0 0.075" rpy="0.0 0.0 0.0"/>
+        <xacro:inertial_box mass="0.5" x="0.3" y="0.3" z="0.15">
+            <origin xyz="0.15 0 0.075" rpy="0 0 0"/>
         </xacro:inertial_box>
     </link>
-    <!-- Left wheel link-->
+    <gazebo reference = "chassis">
+    <material>Gazebo/White</material>
+    </gazebo>
+    <!-- LEFT WHEEL LINK -->
     <joint name="left_wheel_joint" type="continuous">
         <parent link="base_link"/>
         <child link="left_wheel"/>
-        <origin xyz="0.0 0.175 0.0" rpy="-${pi/2} 0.0 0.0"/>
-        <axis xyz="0.0 0.0 1.0"/>
+        <origin xyz="0 0.175 0" rpy="-${pi/2} 0 0" />
+        <axis xyz="0 0 1"/>
     </joint>
     <link name="left_wheel">
@@ -60,14 +71,17 @@
             </geometry>
         </collision>
-        <xacro:inertial_cylinder mass = "0.1" length="0.04" radius="0.05">
-            <origin xyz="0.0 0.0 0.0" rpy="0.0 0.0 0.0"/>
+        <xacro:inertial_cylinder mass="0.1" length="0.04" radius="0.05">
+            <origin xyz="0 0 0" rpy="0 0 0"/>
         </xacro:inertial_cylinder>
     </link>
-    <!-- Right wheel link-->
+    <gazebo reference = "left_wheel">
+    <material>Gazebo/Blue</material>
+    </gazebo>
+    <!-- RIGHT WHEEL LINK -->
     <joint name="right_wheel_joint" type="continuous">
         <parent link="base_link"/>
         <child link="right_wheel"/>
-        <origin xyz="0.0 -0.175 0.0" rpy="${pi/2} 0.0 0.0"/>
-        <axis xyz="0.0 0.0 -1.0"/>
+        <origin xyz="0 -0.175 0" rpy="${pi/2} 0 0" />
+        <axis xyz="0 0 -1"/>
     </joint>
     <link name="right_wheel">
@@ -78,18 +92,21 @@
             <material name="blue"/>
         </visual>
-        <collsion>
+        <collision>
             <geometry>
                 <cylinder radius="0.05" length="0.04"/>
             </geometry>
-        </collsion>
-        <xacro:inertial_cylinder mass = "0.1" length="0.04" radius="0.05">
-            <origin xyz="0.0 0.0 0.0" rpy="0.0 0.0 0.0"/>
+        </collision>
+        <xacro:inertial_cylinder mass="0.1" length="0.04" radius="0.05">
+            <origin xyz="0 0 0" rpy="0 0 0"/>
         </xacro:inertial_cylinder>
     </link>
-    <!-- caster wheel link-->
+    <gazebo reference = "right_wheel">
+    <material>Gazebo/Blue</material>
+    </gazebo>
+    <!-- CASTER WHEEL LINK -->
     <joint name="caster_wheel_joint" type="fixed">
         <parent link="chassis"/>
         <child link="caster_wheel"/>
-        <origin xyz="0.24 0.0 0.0"/>
+        <origin xyz="0.24 0 0"/>
     </joint>
     <link name="caster_wheel">
@@ -105,7 +122,12 @@
             </geometry>
         </collision>
-        <xacro:inertial_sphere mass = "0.1" radius="0.05">
-            <origin xyz="0.0 0.0 0.0" rpy="0.0 0.0 0.0"/>
+        <xacro:inertial_sphere mass="0.1" radius="0.05">
+            <origin xyz="0 0 0" rpy="0 0 0"/>
         </xacro:inertial_sphere>
     </link>
+    <gazebo reference = "caster_wheel">
+        <material>Gazebo/Black</material>
+        <mu1 value="0.005"/>
+        <mu2 value="0.00"/>
+    </gazebo>
 </robot>
